File: Hardware/PCB.brd (EAGLE design)
At the start: 170.2 x 111.2 mm, 103 parts, among them IC1 BD5229G-TR, IC4 XC6220A331MR-G, J1 FH34SRJ-24S-0.5SH_99_, J2 SAMACSYS_PARTS_USB4110-GF-A, J3 QWIIC_RIGHT_ANGLE, J4 112A-TAAR-R03_ATTEND, Q1 20V/4.2A/52mΩ/1.4W, Q2 20V/4.2A/52mΩ/1.4W, Q3 SI1308EDL-T1-GE3, U1 W25Q512JVEIQ, U2 ESP32-C6-WROOM-1-N8, U3 DS3231SN#, U4 MAX17048G+T10

Commit message: Fixed issues
Parts:
- C7: value 10uF -> 10uF
- moved C4_USB 0.30 mm to (155.7, 47.5)
- moved C5_USB 0.30 mm to (155.7, 46.0)
Routing:
- net GND: track 680.4 -> 9.40 mm, vias 18 -> 192
- net 3V3: track 432.2 -> 483.7 mm
- net VBAT: track 30.6 -> 36.0 mm
- net IO/CHANGE: track 82.1 -> 86.9 mm
- net SS_SD: track 64.2 -> 67.8 mm
- net EPD_3V3: track 29.0 -> 30.4 mm
- net SDA: track 194.7 -> 195.9 mm
- net EPD_RST: track 105.4 -> 104.5 mm
- net DP: track 12.1 -> 12.9 mm
- net USB_D-: track 167.4 -> 168.1 mm
