File: Hardware/Schematic.sch (EAGLE design)
At the start: 103 parts, among them IC1 BD5229G-TR, IC4 XC6220A331MR-G, J1 FH34SRJ-24S-0.5SH_99_, J2 SAMACSYS_PARTS_USB4110-GF-A, J3 QWIIC_RIGHT_ANGLE, J4 112A-TAAR-R03_ATTEND, Q1 20V/4.2A/52mΩ/1.4W, Q2 20V/4.2A/52mΩ/1.4W, Q3 SI1308EDL-T1-GE3, U1 W25Q512JVEIQ, U2 ESP32-C6-WROOM-1-N8, U3 DS3231SN#, U4 MAX17048G+T10

Commit message: Fixed issues
Parts:
- C7: value 10uF -> 10uF
Changed lines of the file:
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@@
 <layer number="90" name="Modules" color="5" fill="1" visible="yes" active="yes"/>
 <layer number="91" name="Nets" color="2" fill="1" visible="yes" active="yes"/>
-<layer number="92" name="Busses" color="1" fill="1" visible="no" active="yes"/>
+<layer number="92" name="Busses" color="1" fill="1" visible="yes" active="yes"/>
 <layer number="93" name="Pins" color="2" fill="1" visible="no" active="yes"/>
 <layer number="94" name="Symbols" color="4" fill="1" visible="yes" active="yes"/>
@@
 <part name="GND23" library="DeskAssistant v19 v1" library_urn="urn:adsk.wipprod:fs.file:vf.5HXaHn4GTLqZr9JgB8AkPA" deviceset="GND" device=""/>
 <part name="GND24" library="DeskAssistant v19 v1" library_urn="urn:adsk.wipprod:fs.file:vf.5HXaHn4GTLqZr9JgB8AkPA" deviceset="GND" device=""/>
-<part name="C7" library="DeskAssistant v19 v1" library_urn="urn:adsk.wipprod:fs.file:vf.5HXaHn4GTLqZr9JgB8AkPA" deviceset="ESP32_WROVER_EAGLE-LTSPICE_C" device="C0402" value=" 10uF"/>
+<part name="C7" library="DeskAssistant v19 v1" library_urn="urn:adsk.wipprod:fs.file:vf.5HXaHn4GTLqZr9JgB8AkPA" deviceset="ESP32_WROVER_EAGLE-LTSPICE_C" device="C0402" value="10uF"/>
 <part uuid="2882400048" name="L1" library="DeskAssistant v19 v1" library_urn="urn:adsk.wipprod:fs.file:vf.5HXaHn4GTLqZr9JgB8AkPA" deviceset="744043680" device="IND_4828-WE-TPC_WRE" value="68uH"/>
 <part name="D3" library="DeskAssistant v19 v1" library_urn="urn:adsk.wipprod:fs.file:vf.5HXaHn4GTLqZr9JgB8AkPA" deviceset="MBR0530" device=""/>
@@
 <part name="GND43" library="DeskAssistant v19 v1" library_urn="urn:adsk.wipprod:fs.file:vf.5HXaHn4GTLqZr9JgB8AkPA" deviceset="GND" device=""/>
 <part name="D11" library="DeskAssistant v19 v1" library_urn="urn:adsk.wipprod:fs.file:vf.5HXaHn4GTLqZr9JgB8AkPA" deviceset="PGB1010603MR" device=""/>
-<part name="FRAME1" library="DeskAssistant v19 v1" library_urn="urn:adsk.wipprod:fs.file:vf.5HXaHn4GTLqZr9JgB8AkPA" deviceset="ESP32_WROVER_FRAMES_A3L-LOC" device=""/>
+<part name="FRAME1" library="DeskAssistant v19 v1" library_urn="urn:adsk.wipprod:fs.file:vf.5HXaHn4GTLqZr9JgB8AkPA" deviceset="ESP32_WROVER_FRAMES_A3L-LOC" device="" value="OpenBook Schematic"/>
 <part name="C9" library="DeskAssistant v19 v1" library_urn="urn:adsk.wipprod:fs.file:vf.5HXaHn4GTLqZr9JgB8AkPA" deviceset="ESP32_WROVER_EAGLE-LTSPICE_C" device="C0402" value="100nF"/>
 <part uuid="2882400000" name="J1" library="DeskAssistant v19 v1" library_urn="urn:adsk.wipprod:fs.file:vf.5HXaHn4GTLqZr9JgB8AkPA" deviceset="FH34SRJ-24S-0.5SH_99_" device=""/>
